Commit message: Implemented Gazebo simulator

File: spinning_lidar_description/urdf/hokuyo_ust_20lx.gazebo.xacro (robot description, xacro)
@@ -1,14 +1,11 @@
 <?xml version="1.0"?>
 <robot name="hokuyo_ust_20lx" xmlns:xacro="http://www.ros.org/wiki/xacro">
-    <xacro:macro name="hokuyo_ust_20lx_gazebo" params="name parent *origin ros_topic update_rate ray_count min_angle max_angle">
-		<xacro:hokuyo_utm30lx_model name="${name}">
-			<xacro:insert_block name="origin" />
-		</xacro:hokuyo_utm30lx_model>
-		<gazebo reference="${name}_frame">
-			<sensor type="ray" name="${name}">
+    <xacro:macro name="hokuyo_ust_20lx_gazebo" params="name lidar_link topic update_rate ray_count min_angle max_angle">
+		<gazebo reference="${lidar_link}">
+			<sensor type="ray" name="lidar_sensor">
+				<pose>0 0 0 0 0 0</pose>
+				<visualize>false</visualize>
 				<always_on>true</always_on>
 				<update_rate>${update_rate}</update_rate>
-				<pose>0 0 0 0 0 0</pose>
-				<visualize>false</visualize>
 				<ray>
 					<scan>
@@ -22,5 +19,5 @@
 					<range>
 						<min>0.08</min>
-						<max>30.0</max>
+						<max>60.0</max>
 						<resolution>0.01</resolution>
 					</range>
@@ -32,16 +29,14 @@
 				</ray>
 				<plugin name="gazebo_ros_${name}_controller" filename="libgazebo_ros_laser.so">
-					<topicName>${ros_topic}</topicName>
-					<frameName>${name}_frame</frameName>
+					<topicName>${topic}</topicName>
+					<frameName>${lidar_link}</frameName>
 				</plugin>
 			</sensor>
+			<material>Gazebo/DarkGrey</material>
 		</gazebo>
     </xacro:macro>
-    <xacro:macro name="hokuyo_ust_20lx_gazebo_gpu" params="name parent *origin ros_topic update_rate ray_count min_angle max_angle">
-	    <xacro:hokuyo_utm30lx_model name="${name}">
-	        <xacro:insert_block name="origin" />
-	    </xacro:hokuyo_utm30lx_model>
-    	<gazebo reference="${name}_frame">
-	        <sensor type="gpu_ray" name="${name}">
+    <xacro:macro name="hokuyo_ust_20lx_gazebo_gpu" params="name lidar_link topic update_rate ray_count min_angle max_angle">
+    	<gazebo reference="${lidar_link}">
+	        <sensor type="gpu_ray" name="lidar_sensor_gpu">
 	        	<update_rate>${update_rate}</update_rate>
 	        	<pose>0 0 0 0 0 0</pose>
@@ -58,5 +53,5 @@
 		            <range>
 		            	<min>0.08</min>
-		            	<max>30.0</max>
+		            	<max>60.0</max>
 		            	<resolution>0.01</resolution>
 		            </range>
@@ -68,8 +63,9 @@
 	        	</ray>
 	        	<plugin name="gazebo_ros_${name}_controller" filename="libgazebo_ros_gpu_laser.so">
-		        	<topicName>${ros_topic}</topicName>
-		       		<frameName>${name}_frame</frameName>
+		        	<topicName>${topic}</topicName>
+		       		<frameName>${lidar_link}</frameName>
 	        	</plugin>
 	        </sensor>
+	        <material>Gazebo/DarkGrey</material>
     	</gazebo>
     </xacro:macro>

File: spinning_lidar_description/urdf/rotating_lidar_mount.urdf.xacro (robot description, xacro)
@@ -1,5 +1,5 @@
 <?xml version="1.0"?>
 <robot name="rotating_lidar_mount" xmlns:xacro="http://www.ros.org/wiki/xacro">
-    <!-- <xacro:include filename="$(find spinning_lidar_description)/urdf/Grippers/hokuyo_ust_20lx.gazebo.xacro" /> -->
+    <xacro:include filename="$(find spinning_lidar_description)/urdf/hokuyo_ust_20lx.gazebo.xacro" />
     <xacro:include filename="$(find spinning_lidar_description)/urdf/hokuyo_ust_20lx.urdf.xacro" />
     <xacro:include filename="$(find spinning_lidar_description)/urdf/rotating_lidar_mount.transmission.xacro" />
@@ -8,5 +8,5 @@
     <xacro:macro name="rotating_lidar_mount_macro" params="parent mount_link axis_link lidar_link *origin">
         <link name="${mount_link}">
-            <xacro:inertial_sphere_with_pose mass="0.01" diameter="0.03">
+            <xacro:inertial_sphere_with_pose mass="0.1" diameter="0.03">
                 <origin xyz="0 0 0" rpy="0 0 0"/>
             </xacro:inertial_sphere_with_pose>
@@ -34,5 +34,5 @@
         </joint>
         <link name="${axis_link}">
-            <xacro:inertial_sphere_with_pose mass="0.01" diameter="0.03">
+            <xacro:inertial_sphere_with_pose mass="0.1" diameter="0.03">
                 <origin xyz="0 0 0" rpy="0 0 0"/>
             </xacro:inertial_sphere_with_pose>
@@ -63,4 +63,11 @@
         </joint>
         <xacro:lidar_spin_joint_transmission />
+        <xacro:hokuyo_ust_20lx_gazebo   name="lidar_plugin_gazebo"
+                                        lidar_link="${lidar_link}"
+                                        topic="spinning_lidar/scan"
+                                        update_rate="40.0"
+                                        ray_count="1080"
+                                        min_angle="-270"
+                                        max_angle="270" />
     </xacro:macro>
 </robot>

File: spinning_lidar_description/urdf/spinning_lidar.urdf.xacro (robot description, xacro)
@@ -2,4 +2,5 @@
 <robot name="spinning_hokuyo_utm30lx" xmlns:xacro="http://www.ros.org/wiki/xacro">
     <xacro:include filename="$(find spinning_lidar_description)/urdf/rotating_lidar_mount.urdf.xacro" />
+    <xacro:include filename="$(find spinning_lidar_description)/urdf/spinning_lidar.gazebo" />
     <link name="world"/>
     <xacro:rotating_lidar_mount_macro parent="world" mount_link="laser_mount" axis_link="laser_axis" lidar_link="laser">

Commit message: Implemented IR interrupt in simulation as a plugin. Fixed some bugs in motor control due to yesterda's changes

File: spinning_lidar_description/urdf/hokuyo_ust_20lx.gazebo.xacro (robot description, xacro)
@@ -70,3 +70,10 @@
     	</gazebo>
     </xacro:macro>
+	<gazebo>
+		<plugin name="ir_interrupt_plugin" filename="libir_interrupt_plugin.so">
+ 			<joint>lidar_spin_joint</joint>
+ 			<half_cycle_int>true</half_cycle_int>
+			<angle_tol>0.02</angle_tol>
+		</plugin>
+	</gazebo>
 </robot>
