Commit message: Added description of rotating lidar mount v2 prototype. Changed indentation of all files from tabs to spaces

File: spinning_lidar_description/urdf/spinning_lidar.urdf.xacro (robot description, xacro)
@@ -1,8 +1,12 @@
 <?xml version="1.0"?>
 <robot name="spinning_hokuyo_utm30lx" xmlns:xacro="http://www.ros.org/wiki/xacro">
-    <xacro:include filename="$(find spinning_lidar_description)/urdf/rotating_mounts/rotating_mount_v1.urdf.xacro" />
-    <link name="world"/>
-    <xacro:rotating_mount_v1_macro parent="world" mount_link="laser_mount" axis_link="laser_axis" lidar_link="laser">
-        <origin xyz="0 0 0" rpy="0 0 0" />
-    </xacro:rotating_mount_v1_macro>
+  <xacro:include filename="$(find spinning_lidar_description)/urdf/rotating_mounts/v1/rotating_mount_v1.urdf.xacro" />
+  <xacro:include filename="$(find spinning_lidar_description)/urdf/rotating_mounts/v2/rotating_mount_v2.urdf.xacro" />
+  <link name="world"/>
+<!--   <xacro:rotating_mount_v1_macro parent="world" mount_link="laser_mount" axis_link="laser_axis" lidar_link="laser">
+      <origin xyz="0 0 0" rpy="0 0 0" />
+  </xacro:rotating_mount_v1_macro> -->
+  <xacro:rotating_mount_v2_macro parent="world" imu_link="xsens" mount_link="laser_mount" axis_link="laser_axis" lidar_link="laser">
+      <origin xyz="0 0 0" rpy="0 0 0" />
+  </xacro:rotating_mount_v2_macro>
 </robot>

Commit message: Latest settings to use the new version of the sensor, with IMU

File: spinning_lidar_description/urdf/spinning_lidar.urdf.xacro (robot description, xacro)
@@ -3,9 +3,9 @@
   <xacro:include filename="$(find spinning_lidar_description)/urdf/rotating_mounts/v1/rotating_mount_v1.urdf.xacro" />
   <xacro:include filename="$(find spinning_lidar_description)/urdf/rotating_mounts/v2/rotating_mount_v2.urdf.xacro" />
-  <link name="world"/>
+  <link name="camera"/>
 <!--   <xacro:rotating_mount_v1_macro parent="world" mount_link="laser_mount" axis_link="laser_axis" lidar_link="laser">
       <origin xyz="0 0 0" rpy="0 0 0" />
   </xacro:rotating_mount_v1_macro> -->
-  <xacro:rotating_mount_v2_macro parent="world" imu_link="xsens" mount_link="laser_mount" axis_link="laser_axis" lidar_link="laser">
+  <xacro:rotating_mount_v2_macro parent="camera" imu_link="xsens" mount_link="laser_mount" axis_link="laser_axis" lidar_link="laser">
       <origin xyz="0 0 0" rpy="0 0 0" />
   </xacro:rotating_mount_v2_macro>
