Commit message: Fixed small bug in gazebo laser plugin call

File: spinning_lidar_description/urdf/lidars/hokuyo_ust_20lx.urdf.xacro (robot description, xacro)
@@ -3,4 +3,5 @@
 	<xacro:include filename="$(find hector_xacro_tools)/urdf/inertia_tensors.urdf.xacro" />
 	<xacro:property name="M_PI" value="3.1415926535897931" />
+	<xacro:property name="MAX_ANGLE_SWEEP" value="135.0" />
 	<xacro:macro name="hokuyo_ust_20lx_model" params="name">
 		<link name="${name}">
@@ -27,8 +28,8 @@
 		                                lidar_link="${lidar_link}"
 		                                topic="spinning_lidar/scan"
-		                                update_rate="50.0"
+		                                update_rate="40.0"
 		                                ray_count="1080"
-		                                min_angle="-270.0"
-		                                max_angle="270.0" />
+		                                min_angle="-${MAX_ANGLE_SWEEP}"
+		                                max_angle="${MAX_ANGLE_SWEEP}" />
 	</xacro:macro>
 </robot>
