Commit message: Many changes to the URDF and gazebo subpkg to fix integration issues with ridgeback_yumi

File: spinning_lidar_description/urdf/lidars/hokuyo_ust_20lx.gazebo.xacro (robot description, xacro)
@@ -28,5 +28,5 @@
 					</noise>
 				</ray>
-				<plugin name="gazebo_ros_${name}_controller" filename="libgazebo_ros_laser.so">
+				<plugin name="gazebo_ros_${name}" filename="libgazebo_ros_laser.so">
 					<topicName>${topic}</topicName>
 					<frameName>${lidar_link}</frameName>
@@ -39,7 +39,8 @@
     	<gazebo reference="${lidar_link}">
 	        <sensor type="gpu_ray" name="lidar_sensor_gpu">
-	        	<update_rate>${update_rate}</update_rate>
 	        	<pose>0 0 0 0 0 0</pose>
 	        	<visualize>false</visualize>
+	        	<always_on>true</always_on>
+	        	<update_rate>${update_rate}</update_rate>
 	        	<ray>
 		            <scan>
@@ -62,5 +63,5 @@
 		            </noise>
 	        	</ray>
-	        	<plugin name="gazebo_ros_${name}_controller" filename="libgazebo_ros_gpu_laser.so">
+	        	<plugin name="gazebo_ros_${name}_gpu" filename="libgazebo_ros_gpu_laser.so">
 		        	<topicName>${topic}</topicName>
 		       		<frameName>${lidar_link}</frameName>

File: spinning_lidar_description/urdf/lidars/hokuyo_ust_20lx.urdf.xacro (robot description, xacro)
@@ -1,12 +1,9 @@
 <?xml version="1.0"?>
 <robot name="hokuyo_ust_20lx" xmlns:xacro="http://www.ros.org/wiki/xacro">
+	<xacro:include filename="$(find hector_xacro_tools)/urdf/inertia_tensors.urdf.xacro" />
 	<xacro:property name="M_PI" value="3.1415926535897931" />
 	<xacro:macro name="hokuyo_ust_20lx_model" params="name">
 		<link name="${name}">
-			<inertial>
-				<origin xyz="0 0 0" rpy="0 0 0" />
-				<mass value="0.270" />
-				<inertia ixx="2.632e-4" ixy="0" ixz="0" iyy="2.632e-4" iyz="0" izz="1.62e-4" />
-			</inertial>
+			<xacro:inertial_cuboid mass="0.130" x_length="0.1" y_length="0.1" z_length="0.1"/>
 			<visual>
 				<origin xyz="0 0 0" rpy="0 0 0" />
@@ -21,9 +18,17 @@
 				<origin xyz="0 0 -0.0115" rpy="0 0 0" />
 				<geometry>
-					<box size="0.058 0.058 0.087" />
+					<box size="0.050 0.050 0.070" />
 				<!-- <mesh filename="package://spinning_lidar_description/meshes/LIDAR/hokuyo_ust_10lx.stl"/> -->
 				</geometry>
 			</collision>
 		</link>
+	    <!-- <xacro:hokuyo_ust_20lx_gazebo_gpu   name="hokuyo_ust_20lx_gazebo"  -->
+	    <xacro:hokuyo_ust_20lx_gazebo   name="hokuyo_ust_20lx_gazebo"
+		                                lidar_link="${lidar_link}"
+		                                topic="spinning_lidar/scan"
+		                                update_rate="50.0"
+		                                ray_count="1080"
+		                                min_angle="-270.0"
+		                                max_angle="270.0" />
 	</xacro:macro>
 </robot>

File: spinning_lidar_description/urdf/rotating_mounts/rotating_mount_v1.transmission.xacro (robot description, xacro)
@@ -1,4 +1,4 @@
 <?xml version="1.0"?>
-<robot name="rotating_lidar_mount" xmlns:xacro="http://www.ros.org/wiki/xacro">
+<robot name="rotating_mount_v1" xmlns:xacro="http://www.ros.org/wiki/xacro">
     <xacro:macro name="lidar_spin_joint_transmission">
         <transmission name="lidar_spin_joint_tran">

File: spinning_lidar_description/urdf/rotating_mounts/rotating_mount_v1.urdf.xacro (robot description, xacro)
@@ -1,14 +1,18 @@
 <?xml version="1.0"?>
-<robot name="rotating_lidar_mount" xmlns:xacro="http://www.ros.org/wiki/xacro">
-    <xacro:include filename="$(find spinning_lidar_description)/urdf/hokuyo_ust_20lx.gazebo.xacro" />
-    <xacro:include filename="$(find spinning_lidar_description)/urdf/hokuyo_ust_20lx.urdf.xacro" />
-    <xacro:include filename="$(find spinning_lidar_description)/urdf/rotating_lidar_mount.transmission.xacro" />
+<robot name="rotating_mount_v1" xmlns:xacro="http://www.ros.org/wiki/xacro">
+    <xacro:include filename="$(find spinning_lidar_description)/urdf/lidars/hokuyo_ust_20lx.urdf.xacro" />
+    <xacro:include filename="$(find spinning_lidar_description)/urdf/rotating_mounts/rotating_mount_v1.transmission.xacro" />
+    <xacro:include filename="$(find spinning_lidar_description)/urdf/rotating_mounts/rotating_mount_v1.gazebo" />
     <xacro:include filename="$(find hector_xacro_tools)/urdf/inertia_tensors.urdf.xacro" />
     <xacro:property name="M_PI" value="3.14159265359"/>
-    <xacro:macro name="rotating_lidar_mount_macro" params="parent mount_link axis_link lidar_link *origin">
+    <xacro:macro name="rotating_mount_v1_macro" params="parent mount_link axis_link lidar_link *origin">
+        <link name="${mount_link}_base_link" />
+        <joint name="laser_base_link_to_parent" type="fixed">
+            <parent link="${parent}"/>
+            <child link="${mount_link}_base_link"/>
+            <xacro:insert_block name="origin"/>
+        </joint>
         <link name="${mount_link}">
-            <xacro:inertial_sphere_with_pose mass="0.1" diameter="0.03">
-                <origin xyz="0 0 0" rpy="0 0 0"/>
-            </xacro:inertial_sphere_with_pose>
+            <xacro:inertial_cuboid mass="0.15" x_length="0.4" y_length="0.8" z_length="1.5" />
             <collision name="collision">
                 <origin xyz="0 0 0" rpy="0 0 0"/>
@@ -27,14 +31,12 @@
             </visual>
         </link>
-        <joint name="lidar_mount_root_joint" type="fixed">
-            <xacro:insert_block name="origin"/>
+        <joint name="${mount_link}_base_link_to_mount" type="fixed">
+            <parent link="${mount_link}_base_link"/>
+            <child link="${mount_link}"/>
             <axis xyz="0 0 0"/>
-            <parent link="${parent}"/>
-            <child link="${mount_link}"/>
+            <origin xyz="0 0 0.075" rpy="0 0 0"/>
         </joint>
         <link name="${axis_link}">
-            <xacro:inertial_sphere_with_pose mass="0.1" diameter="0.03">
-                <origin xyz="0 0 0" rpy="0 0 0"/>
-            </xacro:inertial_sphere_with_pose>
+            <xacro:inertial_cuboid mass="0.1" x_length="0.4" y_length="0.8" z_length="1.5"/>
             <visual name="visual">
                 <origin xyz="0 0 0" rpy="0 ${M_PI/2} 0"/>
@@ -53,5 +55,5 @@
             <child link="${axis_link}"/>
             <limit effort="1000" velocity="${2*M_PI}"/>
-            <joint_properties damping="0.0" friction="0.0"/>
+            <joint_properties damping="0.0" />
         </joint>
         <xacro:hokuyo_ust_20lx_model name="${lidar_link}" />
@@ -63,11 +65,5 @@
         </joint>
         <xacro:lidar_spin_joint_transmission />
-        <xacro:hokuyo_ust_20lx_gazebo   name="lidar_plugin_gazebo"
-                                        lidar_link="${lidar_link}"
-                                        topic="spinning_lidar/scan"
-                                        update_rate="40.0"
-                                        ray_count="1080"
-                                        min_angle="-270"
-                                        max_angle="270" />
+        <xacro:rotating_mount_v1_gazebo_macro />
     </xacro:macro>
 </robot>

File: spinning_lidar_description/urdf/spinning_lidar.urdf.xacro (robot description, xacro)
@@ -1,9 +1,8 @@
 <?xml version="1.0"?>
 <robot name="spinning_hokuyo_utm30lx" xmlns:xacro="http://www.ros.org/wiki/xacro">
-    <xacro:include filename="$(find spinning_lidar_description)/urdf/rotating_lidar_mount.urdf.xacro" />
-    <xacro:include filename="$(find spinning_lidar_description)/urdf/spinning_lidar.gazebo" />
+    <xacro:include filename="$(find spinning_lidar_description)/urdf/rotating_mounts/rotating_mount_v1.urdf.xacro" />
     <link name="world"/>
-    <xacro:rotating_lidar_mount_macro parent="world" mount_link="laser_mount" axis_link="laser_axis" lidar_link="laser">
-        <origin xyz="0 0 0.075" rpy="0 0 0" />
-    </xacro:rotating_lidar_mount_macro>
+    <xacro:rotating_mount_v1_macro parent="world" mount_link="laser_mount" axis_link="laser_axis" lidar_link="laser">
+        <origin xyz="0 0 0" rpy="0 0 0" />
+    </xacro:rotating_mount_v1_macro>
 </robot>
