Commit message: Fixed some issues with the URDF, organized files

File: spinning_lidar_description/urdf/lidars/hokuyo_ust_20lx.gazebo.xacro (robot description, xacro)
@@ -1,74 +1,76 @@
 <?xml version="1.0"?>
 <robot name="hokuyo_ust_20lx" xmlns:xacro="http://www.ros.org/wiki/xacro">
-    <xacro:macro name="hokuyo_ust_20lx_gazebo" params="name lidar_link topic update_rate ray_count min_angle max_angle">
-		<gazebo reference="${lidar_link}">
-			<sensor type="ray" name="lidar_sensor">
-				<pose>0 0 0 0 0 0</pose>
-				<visualize>false</visualize>
-				<always_on>true</always_on>
-				<update_rate>${update_rate}</update_rate>
-				<ray>
-					<scan>
-						<horizontal>
-						    <samples>${ray_count}</samples>
-						    <resolution>1</resolution>
-						    <min_angle>${min_angle * M_PI/180}</min_angle>
-						    <max_angle>${max_angle * M_PI/180}</max_angle>
-						</horizontal>
-					</scan>
-					<range>
-						<min>0.08</min>
-						<max>60.0</max>
-						<resolution>0.01</resolution>
-					</range>
-					<noise>
-						<type>gaussian</type>
-						<mean>0.0</mean>
-						<stddev>0.004</stddev>
-					</noise>
-				</ray>
-				<plugin name="gazebo_ros_${name}" filename="libgazebo_ros_laser.so">
-					<topicName>${topic}</topicName>
-					<frameName>${lidar_link}</frameName>
-				</plugin>
-			</sensor>
-			<material>Gazebo/DarkGrey</material>
-		</gazebo>
-    </xacro:macro>
-    <xacro:macro name="hokuyo_ust_20lx_gazebo_gpu" params="name lidar_link topic update_rate ray_count min_angle max_angle">
+  <xacro:macro name="hokuyo_ust_20lx_gazebo" params="name lidar_link topic update_rate ray_count min_angle max_angle gpu">
+    <xacro:if value="${gpu == 'true'}">
     	<gazebo reference="${lidar_link}">
-	        <sensor type="gpu_ray" name="lidar_sensor_gpu">
-	        	<pose>0 0 0 0 0 0</pose>
-	        	<visualize>false</visualize>
-	        	<always_on>true</always_on>
-	        	<update_rate>${update_rate}</update_rate>
-	        	<ray>
-		            <scan>
-		            	<horizontal>
-			                <samples>${ray_count}</samples>
-			                <resolution>1</resolution>
-			                <min_angle>${min_angle * M_PI/180}</min_angle>
-			                <max_angle>${max_angle * M_PI/180}</max_angle>
-		            	</horizontal>
-		            </scan>
-		            <range>
-		            	<min>0.08</min>
-		            	<max>60.0</max>
-		            	<resolution>0.01</resolution>
-		            </range>
-		            <noise>
-		            	<type>gaussian</type>
-		            	<mean>0.0</mean>
-		            	<stddev>0.004</stddev>
-		            </noise>
-	        	</ray>
-	        	<plugin name="gazebo_ros_${name}_gpu" filename="libgazebo_ros_gpu_laser.so">
-		        	<topicName>${topic}</topicName>
-		       		<frameName>${lidar_link}</frameName>
-	        	</plugin>
-	        </sensor>
-	        <material>Gazebo/DarkGrey</material>
+    		<sensor type="ray" name="lidar_sensor">
+    			<pose>0 0 0 0 0 0</pose>
+    			<visualize>false</visualize>
+    			<always_on>true</always_on>
+    			<update_rate>${update_rate}</update_rate>
+    			<ray>
+    				<scan>
+    					<horizontal>
+    				    <samples>${ray_count}</samples>
+    				    <resolution>1</resolution>
+    				    <min_angle>${min_angle * M_PI/180}</min_angle>
+    				    <max_angle>${max_angle * M_PI/180}</max_angle>
+    					</horizontal>
+    				</scan>
+    				<range>
+    					<min>0.08</min>
+    					<max>60.0</max>
+    					<resolution>0.01</resolution>
+    				</range>
+    				<noise>
+    					<type>gaussian</type>
+    					<mean>0.0</mean>
+    					<stddev>0.004</stddev>
+    				</noise>
+    			</ray>
+    			<plugin name="gazebo_ros_${name}" filename="libgazebo_ros_laser.so">
+    				<topicName>${topic}</topicName>
+    				<frameName>${lidar_link}</frameName>
+    			</plugin>
+    		</sensor>
+    		<material>Gazebo/DarkGrey</material>
     	</gazebo>
-    </xacro:macro>
+    </xacro:if>
+    <xacro:unless value="${gpu == 'true'}">
+    	<gazebo reference="${lidar_link}">
+        <sensor type="gpu_ray" name="lidar_sensor_gpu">
+        	<pose>0 0 0 0 0 0</pose>
+        	<visualize>false</visualize>
+        	<always_on>true</always_on>
+        	<update_rate>${update_rate}</update_rate>
+        	<ray>
+            <scan>
+            	<horizontal>
+                <samples>${ray_count}</samples>
+                <resolution>1</resolution>
+                <min_angle>${min_angle * M_PI/180}</min_angle>
+                <max_angle>${max_angle * M_PI/180}</max_angle>
+            	</horizontal>
+            </scan>
+            <range>
+            	<min>0.08</min>
+            	<max>60.0</max>
+            	<resolution>0.01</resolution>
+            </range>
+            <noise>
+            	<type>gaussian</type>
+            	<mean>0.0</mean>
+            	<stddev>0.004</stddev>
+            </noise>
+        	</ray>
+        	<plugin name="gazebo_ros_${name}_gpu" filename="libgazebo_ros_gpu_laser.so">
+          	<topicName>${topic}</topicName>
+         		<frameName>${lidar_link}</frameName>
+        	</plugin>
+        </sensor>
+        <material>Gazebo/DarkGrey</material>
+    	</gazebo>
+    </xacro:unless>
+  </xacro:macro>
 	<gazebo>
 		<plugin name="ir_interrupt_plugin" filename="libir_interrupt_plugin.so">

File: spinning_lidar_description/urdf/lidars/hokuyo_ust_20lx.urdf.xacro (robot description, xacro)
@@ -4,32 +4,32 @@
 	<xacro:property name="M_PI" value="3.1415926535897931" />
 	<xacro:property name="MAX_ANGLE_SWEEP" value="135.0" />
-	<xacro:macro name="hokuyo_ust_20lx_model" params="name">
-		<link name="${name}">
-			<xacro:inertial_cuboid mass="0.130" x_length="0.1" y_length="0.1" z_length="0.1"/>
-			<visual>
-				<origin xyz="0 0 0" rpy="0 0 0" />
-				<geometry>
-					<mesh filename="package://spinning_lidar_description/meshes/LIDAR/hokuyo_ust_10lx.stl" />
-				</geometry>
-		        <material name="Turquoise">
-                    <color rgba="0 1.0 1.0 1" />
-                </material>
-			</visual>
-			<collision>
-				<origin xyz="0 0 -0.0115" rpy="0 0 0" />
-				<geometry>
-					<box size="0.050 0.050 0.070" />
-				<!-- <mesh filename="package://spinning_lidar_description/meshes/LIDAR/hokuyo_ust_10lx.stl"/> -->
-				</geometry>
-			</collision>
-		</link>
-	    <!-- <xacro:hokuyo_ust_20lx_gazebo_gpu   name="hokuyo_ust_20lx_gazebo"  -->
-	    <xacro:hokuyo_ust_20lx_gazebo   name="hokuyo_ust_20lx_gazebo"
-		                                lidar_link="${lidar_link}"
-		                                topic="spinning_lidar/scan"
-		                                update_rate="40.0"
-		                                ray_count="1080"
-		                                min_angle="-${MAX_ANGLE_SWEEP}"
-		                                max_angle="${MAX_ANGLE_SWEEP}" />
-	</xacro:macro>
+  <xacro:macro name="hokuyo_ust_20lx_model" params="name gpu">
+    <link name="${name}">
+      <xacro:inertial_cuboid mass="0.130" x_length="0.1" y_length="0.1" z_length="0.1"/>
+      <visual>
+        <origin xyz="0 0 0" rpy="0 0 0" />
+        <geometry>
+          <mesh filename="package://spinning_lidar_description/meshes/LIDAR/hokuyo_ust_10lx.stl" />
+        </geometry>
+        <material name="Black">
+          <color rgba="0.0 0.0 0.0 1" />
+        </material>
+      </visual>
+      <collision>
+        <origin xyz="0 0 -0.0115" rpy="0 0 0" />
+        <geometry>
+          <box size="0.050 0.050 0.070" />
+        </geometry>
+      </collision>
+    </link>
+    <!-- <xacro:hokuyo_ust_20lx_gazebo_gpu   name="hokuyo_ust_20lx_gazebo"  -->
+    <xacro:hokuyo_ust_20lx_gazebo   name="hokuyo_ust_20lx_gazebo"
+                                    lidar_link="${lidar_link}"
+                                    topic="spinning_lidar/scan"
+                                    update_rate="40.0"
+                                    ray_count="1080"
+                                    min_angle="-${MAX_ANGLE_SWEEP}"
+                                    max_angle="${MAX_ANGLE_SWEEP}"
+                                    gpu="${gpu}" />
+  </xacro:macro>
 </robot>

File: spinning_lidar_description/urdf/rotating_mounts/rotating_mount.transmission.xacro (robot description, xacro)
@@ -1,4 +1,4 @@
 <?xml version="1.0"?>
-<robot name="rotating_mount_v2" xmlns:xacro="http://www.ros.org/wiki/xacro">
+<robot name="rotating_mount" xmlns:xacro="http://www.ros.org/wiki/xacro">
   <xacro:macro name="lidar_spin_joint_transmission">
     <transmission name="lidar_spin_joint_tran">

File: spinning_lidar_description/urdf/rotating_mounts/v1/rotating_mount.urdf.xacro (robot description, xacro)
@@ -1,10 +1,13 @@
 <?xml version="1.0"?>
-<robot name="rotating_mount_v1" xmlns:xacro="http://www.ros.org/wiki/xacro">
+<robot name="rotating_mount" xmlns:xacro="http://www.ros.org/wiki/xacro">
   <xacro:include filename="$(find spinning_lidar_description)/urdf/lidars/hokuyo_ust_20lx.urdf.xacro" />
-  <xacro:include filename="$(find spinning_lidar_description)/urdf/rotating_mounts/v1/rotating_mount_v1.transmission.xacro" />
-  <xacro:include filename="$(find spinning_lidar_description)/urdf/rotating_mounts/v1/rotating_mount_v1.gazebo" />
+  <xacro:include filename="$(find spinning_lidar_description)/urdf/rotating_mounts/rotating_mount.transmission.xacro" />
+  <xacro:include filename="$(find spinning_lidar_description)/urdf/rotating_mounts/v1/rotating_mount.gazebo" />
   <xacro:include filename="$(find hector_xacro_tools)/urdf/inertia_tensors.urdf.xacro" />
   <xacro:property name="M_PI" value="3.14159265359"/>
-  <xacro:macro name="rotating_mount_v1_macro" params="parent mount_link axis_link lidar_link *origin">
+  <material name="grey"><color rgba="0.6 0.6 0.6 1.0" /></material>
+  <material name="orange"><color rgba="1.0 0.54 0.0 1.0" /></material>
+  <material name="white"><color rgba="0.9 0.9 0.9 1.0" /></material>
+  <xacro:macro name="rotating_mount_macro" params="parent mount_link axis_link lidar_link gpu *origin">
     <link name="${mount_link}_base_link" />
     <joint name="laser_base_link_to_parent" type="fixed">
@@ -26,7 +29,5 @@
           <box size="0.04 0.08 0.15"/>
         </geometry>
-        <material name="Grey">
-          <color rgba="0.6 0.6 0.6 1"/>
-        </material>
+        <material name="grey" />
       </visual>
     </link>
@@ -44,7 +45,5 @@
           <cylinder length="0.035" radius="0.02"/>
         </geometry>
-        <material name="Grey">
-          <color rgba="0.6 0.6 0.6 1"/>
-        </material>
+        <material name="grey" />
       </visual>
     </link>
@@ -57,5 +56,5 @@
       <joint_properties damping="0.0" />
     </joint>
-    <xacro:hokuyo_ust_20lx_model name="${lidar_link}" />
+    <xacro:hokuyo_ust_20lx_model name="${lidar_link}" gpu="${gpu}"/>
     <joint name="lidar_offset_joint" type="fixed">
       <origin xyz="0.035 0 0.025" rpy="0 0 0"/>
@@ -65,5 +64,5 @@
     </joint>
     <xacro:lidar_spin_joint_transmission />
-    <xacro:rotating_mount_v1_gazebo_macro />
+    <xacro:rotating_mount_gazebo_macro />
   </xacro:macro>
 </robot>

File: spinning_lidar_description/urdf/rotating_mounts/v2/rotating_mount.urdf.xacro (robot description, xacro)
@@ -1,10 +1,13 @@
 <?xml version="1.0"?>
-<robot name="rotating_mount_v2" xmlns:xacro="http://www.ros.org/wiki/xacro">
+<robot name="rotating_mount" xmlns:xacro="http://www.ros.org/wiki/xacro">
   <xacro:include filename="$(find spinning_lidar_description)/urdf/lidars/hokuyo_ust_20lx.urdf.xacro" />
-  <xacro:include filename="$(find spinning_lidar_description)/urdf/rotating_mounts/v2/rotating_mount_v2.transmission.xacro" />
-  <xacro:include filename="$(find spinning_lidar_description)/urdf/rotating_mounts/v2/rotating_mount_v2.gazebo" />
+  <xacro:include filename="$(find spinning_lidar_description)/urdf/rotating_mounts/rotating_mount.transmission.xacro" />
+  <xacro:include filename="$(find spinning_lidar_description)/urdf/rotating_mounts/v2/rotating_mount.gazebo" />
   <xacro:include filename="$(find hector_xacro_tools)/urdf/inertia_tensors.urdf.xacro" />
   <xacro:property name="M_PI" value="3.14159265359"/>
-  <xacro:macro name="rotating_mount_v2_macro" params="parent imu_link mount_link axis_link lidar_link *origin">
+  <material name="grey"><color rgba="0.6 0.6 0.6 1.0" /></material>
+  <material name="orange"><color rgba="1.0 0.54 0.0 1.0" /></material>
+  <material name="white"><color rgba="0.9 0.9 0.9 1.0" /></material>
+  <xacro:macro name="rotating_mount_macro" params="parent imu_link mount_link axis_link lidar_link gpu *origin">
     <link name="${mount_link}_base_link" />
     <joint name="laser_base_link_to_parent" type="fixed">
@@ -26,7 +29,5 @@
           <box size="0.04 0.08 0.15"/>
         </geometry>
-        <material name="Grey">
-          <color rgba="0.6 0.6 0.6 1"/>
-        </material>
+        <material name="grey" />
       </visual>
     </link>
@@ -50,7 +51,5 @@
           <mesh scale="0.001 0.001 0.001" filename="package://spinning_lidar_description/meshes/IMU/xsens-mti30.stl" />
         </geometry>
-        <material name="Orange">
-          <color rgba="1.0 0.54 0 1"/>
-        </material>
+        <material name="orange" />
       </visual>
     </link>
@@ -68,7 +67,5 @@
           <cylinder length="0.035" radius="0.02"/>
         </geometry>
-        <material name="Grey">
-          <color rgba="0.6 0.6 0.6 1"/>
-        </material>
+        <material name="grey" />
       </visual>
     </link>
@@ -81,5 +78,5 @@
       <joint_properties damping="0.0" />
     </joint>
-    <xacro:hokuyo_ust_20lx_model name="${lidar_link}" />
+    <xacro:hokuyo_ust_20lx_model name="${lidar_link}" gpu="${gpu}"/>
     <joint name="lidar_offset_joint" type="fixed">
       <origin xyz="0.035 0 0.025" rpy="0 0 0"/>
@@ -89,5 +86,5 @@
     </joint>
     <xacro:lidar_spin_joint_transmission />
-    <xacro:rotating_mount_v2_gazebo_macro imu_link="${imu_link}"/>
+    <xacro:rotating_mount_gazebo_macro imu_link="${imu_link}"/>
   </xacro:macro>
 </robot>

File: spinning_lidar_description/urdf/spinning_lidar.urdf.xacro (robot description, xacro)
@@ -1,12 +1,13 @@
 <?xml version="1.0"?>
 <robot name="spinning_hokuyo_utm30lx" xmlns:xacro="http://www.ros.org/wiki/xacro">
-  <xacro:include filename="$(find spinning_lidar_description)/urdf/rotating_mounts/v1/rotating_mount_v1.urdf.xacro" />
-  <xacro:include filename="$(find spinning_lidar_description)/urdf/rotating_mounts/v2/rotating_mount_v2.urdf.xacro" />
+  <!-- Includes -->
+  <xacro:include filename="$(find spinning_lidar_description)/urdf/rotating_mounts/v2/rotating_mount.urdf.xacro" />
+  <!-- GPU acceleration -->
+  <xacro:arg name="gpu" default="false"/>
+  <xacro:property name="gpu" value="$(arg gpu)" />
+  <!-- Robot tree construction -->
   <link name="camera"/>
-<!--   <xacro:rotating_mount_v1_macro parent="world" mount_link="laser_mount" axis_link="laser_axis" lidar_link="laser">
-      <origin xyz="0 0 0" rpy="0 0 0" />
-  </xacro:rotating_mount_v1_macro> -->
-  <xacro:rotating_mount_v2_macro parent="camera" imu_link="xsens" mount_link="laser_mount" axis_link="laser_axis" lidar_link="laser">
-      <origin xyz="0 0 0" rpy="0 0 0" />
-  </xacro:rotating_mount_v2_macro>
+  <xacro:rotating_mount_macro parent="camera" imu_link="xsens" mount_link="laser_mount" axis_link="laser_axis" lidar_link="laser" gpu="${gpu}">
+    <origin xyz="0 0 0" rpy="0 0 0" />
+  </xacro:rotating_mount_macro>
 </robot>

Commit message: A few changes to make the pkg compatible with ROS Melodic and Gazebo 9. Tuned IR int plugin

File: spinning_lidar_description/urdf/lidars/hokuyo_ust_20lx.gazebo.xacro (robot description, xacro)
@@ -2,81 +2,82 @@
 <robot name="hokuyo_ust_20lx" xmlns:xacro="http://www.ros.org/wiki/xacro">
   <xacro:macro name="hokuyo_ust_20lx_gazebo" params="name lidar_link topic update_rate ray_count min_angle max_angle gpu">
-    <xacro:if value="${gpu == 'true'}">
-    	<gazebo reference="${lidar_link}">
-    		<sensor type="ray" name="lidar_sensor">
-    			<pose>0 0 0 0 0 0</pose>
-    			<visualize>false</visualize>
-    			<always_on>true</always_on>
-    			<update_rate>${update_rate}</update_rate>
-    			<ray>
-    				<scan>
-    					<horizontal>
-    				    <samples>${ray_count}</samples>
-    				    <resolution>1</resolution>
-    				    <min_angle>${min_angle * M_PI/180}</min_angle>
-    				    <max_angle>${max_angle * M_PI/180}</max_angle>
-    					</horizontal>
-    				</scan>
-    				<range>
-    					<min>0.08</min>
-    					<max>60.0</max>
-    					<resolution>0.01</resolution>
-    				</range>
-    				<noise>
-    					<type>gaussian</type>
-    					<mean>0.0</mean>
-    					<stddev>0.004</stddev>
-    				</noise>
-    			</ray>
-    			<plugin name="gazebo_ros_${name}" filename="libgazebo_ros_laser.so">
-    				<topicName>${topic}</topicName>
-    				<frameName>${lidar_link}</frameName>
-    			</plugin>
-    		</sensor>
-    		<material>Gazebo/DarkGrey</material>
-    	</gazebo>
-    </xacro:if>
     <xacro:unless value="${gpu == 'true'}">
-    	<gazebo reference="${lidar_link}">
-        <sensor type="gpu_ray" name="lidar_sensor_gpu">
-        	<pose>0 0 0 0 0 0</pose>
-        	<visualize>false</visualize>
-        	<always_on>true</always_on>
-        	<update_rate>${update_rate}</update_rate>
-        	<ray>
+      <gazebo reference="${lidar_link}">
+        <sensor type="ray" name="lidar_sensor">
+          <pose>0 0 0 0 0 0</pose>
+          <visualize>false</visualize>
+          <always_on>true</always_on>
+          <update_rate>${update_rate}</update_rate>
+          <ray>
             <scan>
-            	<horizontal>
-                <samples>${ray_count}</samples>
-                <resolution>1</resolution>
-                <min_angle>${min_angle * M_PI/180}</min_angle>
-                <max_angle>${max_angle * M_PI/180}</max_angle>
-            	</horizontal>
+              <horizontal>
+              <samples>${ray_count}</samples>
+              <resolution>1</resolution>
+              <min_angle>${min_angle * M_PI/180}</min_angle>
+              <max_angle>${max_angle * M_PI/180}</max_angle>
+              </horizontal>
             </scan>
             <range>
-            	<min>0.08</min>
-            	<max>60.0</max>
-            	<resolution>0.01</resolution>
+              <min>0.08</min>
+              <max>60.0</max>
+              <resolution>0.01</resolution>
             </range>
             <noise>
-            	<type>gaussian</type>
-            	<mean>0.0</mean>
-            	<stddev>0.004</stddev>
+              <type>gaussian</type>
+              <mean>0.0</mean>
+              <stddev>0.004</stddev>
             </noise>
-        	</ray>
-        	<plugin name="gazebo_ros_${name}_gpu" filename="libgazebo_ros_gpu_laser.so">
-          	<topicName>${topic}</topicName>
-         		<frameName>${lidar_link}</frameName>
-        	</plugin>
+          </ray>
+          <plugin name="gazebo_ros_${name}" filename="libgazebo_ros_laser.so">
+            <topicName>${topic}</topicName>
+            <frameName>${lidar_link}</frameName>
+          </plugin>
         </sensor>
         <material>Gazebo/DarkGrey</material>
-    	</gazebo>
+      </gazebo>
     </xacro:unless>
+    <xacro:if value="${gpu == 'true'}">
+      <gazebo reference="${lidar_link}">
+      <sensor type="gpu_ray" name="lidar_sensor_gpu">
+        <pose>0 0 0 0 0 0</pose>
+        <visualize>false</visualize>
+        <always_on>true</always_on>
+        <update_rate>${update_rate}</update_rate>
+        <ray>
+        <scan>
+          <horizontal>
+          <samples>${ray_count}</samples>
+          <resolution>1</resolution>
+          <min_angle>${min_angle * M_PI/180}</min_angle>
+          <max_angle>${max_angle * M_PI/180}</max_angle>
+          </horizontal>
+        </scan>
+        <range>
+          <min>0.08</min>
+          <max>60.0</max>
+          <resolution>0.01</resolution>
+        </range>
+        <noise>
+          <type>gaussian</type>
+          <mean>0.0</mean>
+          <stddev>0.004</stddev>
+        </noise>
+        </ray>
+        <plugin name="gazebo_ros_${name}_gpu" filename="libgazebo_ros_gpu_laser.so">
+          <topicName>${topic}</topicName>
+          <frameName>${lidar_link}</frameName>
+        </plugin>
+      </sensor>
+      <material>Gazebo/DarkGrey</material>
+      </gazebo>
+    </xacro:if>
   </xacro:macro>
-	<gazebo>
-		<plugin name="ir_interrupt_plugin" filename="libir_interrupt_plugin.so">
- 			<joint>lidar_spin_joint</joint>
- 			<half_cycle_int>true</half_cycle_int>
-			<angle_tol>0.02</angle_tol>
-		</plugin>
-	</gazebo>
+  <gazebo>
+    <plugin name="ir_interrupt_plugin" filename="libir_interrupt_plugin.so">
+      <joint>lidar_spin_joint</joint>
+      <frame_id>laser_mount</frame_id>
+      <half_cycle_int>true</half_cycle_int>
+      <angle_tol>0.002</angle_tol>
+    </plugin>
+  </gazebo>
 </robot>

File: spinning_lidar_description/urdf/spinning_lidar.urdf.xacro (robot description, xacro)
@@ -7,6 +7,6 @@
   <xacro:property name="gpu" value="$(arg gpu)" />
   <!-- Robot tree construction -->
-  <link name="camera"/>
-  <xacro:rotating_mount_macro parent="camera" imu_link="xsens" mount_link="laser_mount" axis_link="laser_axis" lidar_link="laser" gpu="${gpu}">
+  <link name="world"/>
+  <xacro:rotating_mount_macro parent="world" imu_link="xsens" mount_link="laser_mount" axis_link="laser_axis" lidar_link="laser" gpu="${gpu}">
     <origin xyz="0 0 0" rpy="0 0 0" />
   </xacro:rotating_mount_macro>
